File: Simulation/MPS Stimulator/MPSStimulator.sch (KiCad schematic (older format))
At the start: 87 parts, among them Q10 BCY58, Q11 BCY58, Q12 BCY58, Q3 BCY58, Q4 BCY58, Q5 BCY58, Q6 BCY58, Q7 BCY58, Q8 BCY58, Q9 BCY58

Commit message: Generates a 0-5V output.
Parts:
- removed C1, C2: 2.2n, Right D Line, symbol Device:C
- removed C7: 470n, Right D Line, symbol Device:C
- removed C8: 33n, Right D Line, symbol Device:C
- removed D13, D6, D7, D8, D9: DIODE, symbol Simulation_SPICE:DIODE
- removed Q3, Q4, Q5, Q6, Q7, Q9: BCY58, Package_TO_SOT_THT:TO-92_Inline, symbol Transistor_BJT:BC547
- removed R15, R16, R17, R18, R19, R20, R21, R22: 3k, Upper Center K, symbol Device:R_US
- removed R28, R29: 300, Upper Center K, symbol Device:R_US
- removed R32, R33, R34, R35: 180k, Upper Center K, symbol Device:R_US
- removed R37, R38, R39, R40: 1k, Upper Center K, symbol Device:R_US
- removed R43, R44, R45, R46: 10k, Upper Center K, symbol Device:R_US
- removed R47, R51: 2k, Upper Center K, symbol Device:R_US
- removed R49, R52: 5k1, Upper Center K, symbol Device:R_US
- removed R54: 1k3, Upper Center K, symbol Device:R_US
- removed R55: 27k, Upper Center K, symbol Device:R_US
- removed R56: 130k, Upper Center K, symbol Device:R_US
- removed R57: 20k, Upper Center K, symbol Device:R_US
- removed R58, R59: 36k, Upper Center K, symbol Device:R_US
- removed V3, V4, V5, V6: VPULSE, symbol Simulation_SPICE:VPULSE
- added Q1: BCY58, Package_TO_SOT_THT:TO-92_Inline, symbol Transistor_BJT:BC547
- added R1: 2k, Upper Center K, symbol Device:R_US
- added R2: 20k, Upper Center K, symbol Device:R_US
- added R3, R4, R5: 10k, Upper Center K, symbol Device:R_US
- added V8: VPULSE, symbol Simulation_SPICE:VPULSE
Connections:
- net 0: now also Q1.3 (E), R3.2, R5.1, V8.2
- net AUX1-10V: now also R1.2
- net BASE_PULSE: now also R2.1
- net INT-7 renamed IN
- net IN: now also V8.1
- new net: Q1.1 (C), R1.1, R4.2
- new net: Q1.2 (B), R2.2, R3.1
- new net OUT: R4.1, R5.2
Other:
- note added: ".model DIODE D\n.model BCY58 npn\n.model BSX95 npn\n.model AUY21 pnp\n\n.tran 0.05ms 100ms 89m\n\n.control\nrun\nrusage\nset filetype=ascii\nset color0=white\nset xbrushwidth=5\n\n*write "C:\Users\andy\OneDrive\Documents\MPS Tune-o-Matic\trunk\Simulation\Pressure Loop\PressureLoop.out" "V(BASE_PULSE)" "V(INT-7)"\nplot "V(IN)"+0 "V(OUT)"+0\n\n.endc\n"
- note removed: ".model DIODE D\n.model BCY58 npn\n.model BSX95 npn\n.model AUY21 pnp\n\n.tran 0.05ms 92ms 89m\n\n.control\nrun\nrusage\nset filetype=ascii\nset color0=white\nset xbrushwidth=5\n\n* pulse generator 0.05ms 400ms 100ms\n*plot "V(E13-PG)" "V(E22-PG)"+4 "V(E14-PG)"+8 "V(E21-PG)"+12\n\n* flip-flip and NOR output 0.05ms 400ms 100ms\n*plot "V(INT-7)"+0 "V(E13-PG)"+2 "V(E22-PG)"+6 "V(E14-PG)"+10 "V(E21-PG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"
- note removed: "Engine speed of 666.67 RPM\n= 333.35 RPM at distributor\n= 333.35 / 60 = 5.56 rotations per second at distributor\n1 / 5.56 = 180ms per rotation\n120 degrees of dwell = 180ms / 3 = 60ms\n"
- note removed: "I"
- note removed: "II"
- note removed: "III"
- note removed: "IV"
- moved on the sheet: C4, C5, C9, D14, D15, D16, D4, D5, Q10, Q11, Q12, Q8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

Commit message: Completed stimulator. Added example waveforms.
Parts:
- removed R60: 200, Upper Center K, symbol Device:R_US
- added R7: 1k, Upper Center K, symbol Device:R_US
- added RV1: 5k, symbol Device:Varistor
- added RV2: 1k, symbol Device:Varistor
- R5: value 10k -> 12k
- V7: value 4 -> 5; Spice_Model dc(4.0) -> dc(5.0)
Connections:
- net 0: now also R7.1, RV2.2
- net E1-T1: now also RV2.1
- net E10-MPS: now also R7.2, RV1.2; no longer V7.1
- new net INT-6: RV1.1, V7.1
Other:
- note added: ".model DIODE D\n.model BCY58 npn\n.model BSX95 npn\n.model AUY21 pnp\n\n.tran 0.05ms 100ms 89m\n\n.control\nrun\nrusage\nset filetype=ascii\nset color0=white\nset xbrushwidth=5\n\n*write "C:\Users\andy\OneDrive\Documents\MPS Tune-o-Matic\trunk\Simulation\Pressure Loop\PressureLoop.out" "V(BASE_PULSE)" "V(INT-7)"\nplot "V(IN)"+0 "V(BASE_PULSE)"+6 "V(OUT)"+33\n\n.endc\n"
- note removed: ".model DIODE D\n.model BCY58 npn\n.model BSX95 npn\n.model AUY21 pnp\n\n.tran 0.05ms 100ms 89m\n\n.control\nrun\nrusage\nset filetype=ascii\nset color0=white\nset xbrushwidth=5\n\n*write "C:\Users\andy\OneDrive\Documents\MPS Tune-o-Matic\trunk\Simulation\Pressure Loop\PressureLoop.out" "V(BASE_PULSE)" "V(INT-7)"\nplot "V(IN)"+0 "V(OUT)"+0\n\n.endc\n"
Changed lines of the file:
@@
 	8850 7700 9100 7700
 Connection ~ 9100 7700
-$Comp
-L Device:R_US R60
-U 1 1 6280EC00
-P 8050 8100
-F 0 "R60" V 7950 8000 50  0000 L CNN
-F 1 "200" V 8150 8000 50  0000 L CNN
-F 2 "Upper Center K" V 8090 8090 50  0001 C CNN
-F 3 "~" H 8050 8100 50  0001 C CNN
-F 4 "O Bk Br Gd = 300Ω ±5%" H 8050 8100 50  0001 C CNN "Notes"
-	1    8050 8100
-	-1   0    0    1
-$EndComp
 Wire Wire Line
 	8550 7700 8050 7700
@@
 P 1300 4250
 F 0 "V7" H 1430 4341 50  0000 L CNN
-F 1 "4" H 1430 4250 50  0000 L CNN
+F 1 "5" H 1430 4250 50  0000 L CNN
 F 2 "" H 1300 4250 50  0001 C CNN
 F 3 "~" H 1300 4250 50  0001 C CNN
 F 4 "Y" H 1300 4250 50  0001 L CNN "Spice_Netlist_Enabled"
 F 5 "V" H 1300 4250 50  0001 L CNN "Spice_Primitive"
-F 6 "dc(4.0)" H 1430 4159 50  0000 L CNN "Spice_Model"
+F 6 "dc(5.0)" H 1430 4159 50  0000 L CNN "Spice_Model"
 	1    1300 4250
 	1    0    0    -1
@@
 Wire Wire Line
 	1300 4050 1300 3000
-Connection ~ 10050 8850
 Wire Wire Line
 	10050 8500 10050 8850
@@
 Text GLabel 9950 8500 0    50   Input ~ 0
 E10-MPS
-Text GLabel 9950 8850 0    50   Input ~ 0
+Text GLabel 8800 8300 0    50   Input ~ 0
 INT-6
 Wire Wire Line
-	9950 8850 10050 8850
-Wire Wire Line
-	8050 9700 12700 9700
+	8050 9700 9100 9700
 Connection ~ 12700 9700
 Wire Wire Line
@@
 Lower voltage = richer
 Text Notes 1350 9300 0    50   ~ 0
-.model DIODE D\n.model BCY58 npn\n.model BSX95 npn\n.model AUY21 pnp\n\n.tran 0.05ms 100ms 89m\n\n.control\nrun\nrusage\nset filetype=ascii\nset color0=white\nset xbrushwidth=5\n\n*write "C:\Users\andy\OneDrive\Documents\MPS Tune-o-Matic\trunk\Simulation\Pressure Loop\PressureLoop.out" "V(BASE_PULSE)" "V(INT-7)"\nplot "V(IN)"+0 "V(OUT)"+0\n\n.endc\n
+.model DIODE D\n.model BCY58 npn\n.model BSX95 npn\n.model AUY21 pnp\n\n.tran 0.05ms 100ms 89m\n\n.control\nrun\nrusage\nset filetype=ascii\nset color0=white\nset xbrushwidth=5\n\n*write "C:\Users\andy\OneDrive\Documents\MPS Tune-o-Matic\trunk\Simulation\Pressure Loop\PressureLoop.out" "V(BASE_PULSE)" "V(INT-7)"\nplot "V(IN)"+0 "V(BASE_PULSE)"+6 "V(OUT)"+33\n\n.endc\n
 Wire Wire Line
 	15200 3900 14150 3900
@@
 P 18100 8350
 F 0 "R4" H 17950 8400 50  0000 L CNN
-F 1 "10k" H 17950 8300 50  0000 L CNN
+F 1 "10k" H 17900 8300 50  0000 L CNN
 F 2 "Upper Center K" V 18140 8340 50  0001 C CNN
 F 3 "~" H 18100 8350 50  0001 C CNN
@@
 P 18100 9050
 F 0 "R5" H 17950 9100 50  0000 L CNN
-F 1 "10k" H 17950 9000 50  0000 L CNN
+F 1 "12k" H 17900 9000 50  0000 L CNN
 F 2 "Upper Center K" V 18140 9040 50  0001 C CNN
 F 3 "~" H 18100 9050 50  0001 C CNN
@@
 Wire Wire Line
 	18100 8700 18100 8500
+Connection ~ 9100 9700
+Wire Wire Line
+	9100 9700 12700 9700
+Wire Wire Line
+	9100 8300 8800 8300
+Wire Wire Line
+	9100 9350 9100 9700
+Wire Wire Line
+	9100 8400 9100 8300
+Connection ~ 10050 8850
+Wire Wire Line
+	9100 8850 10050 8850
+Wire Wire Line
+	9100 8850 9100 9050
+Connection ~ 9100 8850
+Wire Wire Line
+	9100 8700 9100 8850
+$Comp
+L Device:R_US R7
+U 1 1 62182801
+P 9100 9200
+F 0 "R7" V 9000 9100 50  0000 L CNN
+F 1 "1k" V 9200 9100 50  0000 L CNN
+F 2 "Upper Center K" V 9140 9190 50  0001 C CNN
+F 3 "~" H 9100 9200 50  0001 C CNN
+F 4 "O Bk Br Gd = 300Ω ±5%" H 9100 9200 50  0001 C CNN "Notes"
+	1    9100 9200
+	-1   0    0    1
+$EndComp
+$Comp
+L Device:Varistor RV1
+U 1 1 621ABE67
+P 9100 8550
+F 0 "RV1" H 9203 8596 50  0000 L CNN
+F 1 "5k" H 9203 8505 50  0000 L CNN
+F 2 "" V 9030 8550 50  0001 C CNN
+F 3 "~" H 9100 8550 50  0001 C CNN
+	1    9100 8550
+	1    0    0    -1
+$EndComp
+$Comp
+L Device:Varistor RV2
+U 1 1 621AEB7C
+P 8050 8100
+F 0 "RV2" H 8153 8146 50  0000 L CNN
+F 1 "1k" H 8153 8055 50  0000 L CNN
+F 2 "" V 7980 8100 50  0001 C CNN
+F 3 "~" H 8050 8100 50  0001 C CNN
+	1    8050 8100
+	1    0    0    -1
+$EndComp
 $EndSCHEMATC
