File: PCB/MPS Driver.sch (KiCad schematic (older format))
At the start: 12 parts

Commit message: WIP
Parts:
- removed Q? (x2): MMBT2222ALT1G, Package_TO_SOT_SMD:SOT-23, symbol Transistor_BJT:MMBT3904
- removed Q? (x2): MMBT3906LT1G, Package_TO_SOT_SMD:SOT-23, symbol Device:Q_PNP_BEC
- removed R? (x4): 1k, Resistor_SMD:R_0805_2012Metric, symbol Device:R
- removed R? (x4): 10k, Resistor_SMD:R_0805_2012Metric, symbol Device:R
- added C?: 1n0, Capacitor_SMD:C_0603_1608Metric, symbol Device:C
- added C? (x2): 6n8, Capacitor_SMD:C_0603_1608Metric, symbol Device:C
- added D? (x5): D, Diode_SMD:D_SOD-523, symbol Device:D
- added R?: 240, Resistor_SMD:R_0603_1608Metric, symbol Device:R
- added R?: 1k2, Resistor_SMD:R_0603_1608Metric, symbol Device:R
- added R?: 510, Resistor_SMD:R_0805_2012Metric, symbol Device:R
- added R?: 2k2, Resistor_SMD:R_0603_1608Metric, symbol Device:R
- added R?: 2K, Resistor_SMD:R_0603_1608Metric, symbol Device:R
- added R?: 300, Resistor_SMD:R_0603_1608Metric, symbol Device:R
- added R?: 1K, Resistor_SMD:R_0603_1608Metric, symbol Device:R
- added R?: 2k4, Resistor_SMD:R_0603_1608Metric, symbol Device:R
- added R?: 180K, Resistor_SMD:R_0603_1608Metric, symbol Device:R
- added R? (x2): 68K, Resistor_SMD:R_0603_1608Metric, symbol Device:R
- added R? (x2): 130K, Resistor_SMD:R_0603_1608Metric, symbol Device:R
- added R?: 100K, Resistor_SMD:R_0603_1608Metric, symbol Device:R
- added T? (x2): PZT2222A,115, Package_TO_SOT_SMD:SOT-223-3_TabPin2, symbol Transistor_BJT:2SD1047
Connections:
- net ECU_AIRTEMP: now also R?.2
- net GND: now also R?.2, R?.2, R?.2, T?.3 (E), T?.3 (E)
- net MPS-15: now also R?.1, R?.2
- net MPS-7: now also R?.2, T?.2 (C)
- net MPS-8: now also D?.1 (K)
- new net: D?.2 (A), D?.2 (A), D?.2 (A), D?.2 (A), R?.2
- new net: D?.2 (A), R?.1, R?.2
- new net: D?.1 (K), R?.2
- new net: C?.2, R?.1
- new net: D?.1 (K), R?.1, R?.2, T?.1 (B)
- new net: C?.1, R?.2, T?.1 (B)
- new net: C?.1, D?.1 (K), R?.1, R?.2 (x2)
- new net +10V: C?.2, R?.1, R?.1, R?.1, R?.1, R?.1, R?.1, R?.1
- new net ENABLE_II_IV_12V: C?.2
- new net SPEED_SENSOR_PULSE_12V: R?.1, R?.2, T?.2 (C)
Other:
- note added: "7 and 8 are MPS coil outputs"
