File: Simulation/Pressure Loop/PressureLoop.sch (KiCad schematic (older format))
At the start: 49 parts, among them Q1 BCY58, Q2 BCY58, Q3 BCY58, Q4 BCY58, Q5 BCY58, Q6 BCY58, Q7 BCY58, Q8 BCY58

Commit message: Wprking on simulation of pressure loop.
Parts:
- added C3, C8: 33n, Right D Line, symbol Device:C
- added C4, C5: 6.8n, Right D Line, symbol Device:C
- added C6, C7: 470n, Right D Line, symbol Device:C
- added C9: 1.0n, Right D Line, symbol Device:C
- added D10, D11, D12, D13, D14, D15, D16, D2, D3, D4, D5, D9: DIODE, symbol Simulation_SPICE:DIODE
- added L1: 395mH, symbol pspice:INDUCTOR
- added L2: 792mH, symbol pspice:INDUCTOR
- added Q1, Q11, Q12: BCY58, Package_TO_SOT_THT:TO-92_Inline, symbol Transistor_BJT:BC547
- added Q2: AUY21, symbol Device:Q_PNP_CBE
- added R1, R23: 100k, Upper Center K, symbol Device:R_US
- added R10: 510k, Upper Center K, symbol Device:R_US
- added R11, R7: 22k, Upper Center K, symbol Device:R_US
- added R12, R26, R31: 68k, Upper Center K, symbol Device:R_US
- added R13, R14, R24: 10k, Upper Center K, symbol Device:R_US
- added R2, R4: 1k5, Upper Center K, symbol Device:R_US
- added R25, R30, R56: 130k, Upper Center K, symbol Device:R_US
- added R27: 5k6, Upper Center K, symbol Device:R_US
- added R3: 100, Upper Center K, symbol Device:R_US
- added R36: 9k1, Upper Center K, symbol Device:R_US
- added R41: 270k, Upper Center K, symbol Device:R_US
- added R42: 75k, Upper Center K, symbol Device:R_US
- added R5: 15k, Upper Center K, symbol Device:R_US
- added R54: 1k3, Upper Center K, symbol Device:R_US
- added R55: 27k, Upper Center K, symbol Device:R_US
- added R57: 20k, Upper Center K, symbol Device:R_US
- added R58, R59: 36k, Upper Center K, symbol Device:R_US
- added R6, R67: 2k4, Upper Center K, symbol Device:R_US
- added R60, R61: 240, Upper Center K, symbol Device:R_US
- added R62: 1k2, Upper Center K, symbol Device:R_US
- added R63: 2k2, Upper Center K, symbol Device:R_US
- added R64: 510, Upper Center K, symbol Device:R_US
- added R65: 180k, Upper Center K, symbol Device:R_US
- added R66: 2k, Upper Center K, symbol Device:R_US
- added R68: 300, Upper Center K, symbol Device:R_US
- added R69: 1k, Upper Center K, symbol Device:R_US
- added R70: 90.7, Upper Center K, symbol Device:R_US
- added R71: 340.4, Upper Center K, symbol Device:R_US
- added R8: 4k8, Upper Center K, symbol Device:R_US
- added R9: 56k, Upper Center K, symbol Device:R_US
- added V1: 10, symbol Simulation_SPICE:VDC
- added V7: 2, symbol Simulation_SPICE:VDC
- added VBOGUS1: 0, symbol Simulation_SPICE:VDC
- C1, C2: value 2n2 -> 2.2n
- renumbered D4 to D1, D1 to D6, D2 to D7, D3 to D8, Q8 to Q10, Q1 to Q3, Q2 to Q4, Q3 to Q7, Q7 to Q8, Q4 to Q9, R1 to R15, R2 to R16, R3 to R17, R4 to R18, R16 to R19, R17 to R20, R18 to R21, R19 to R22, R5 to R28, R20 to R29, R6 to R32, R7 to R33, R21 to R34, R22 to R35, R8 to R37, R9 to R38, R23 to R39, R24 to R40, R10 to R43, R11 to R44, R25 to R45, R26 to R46, R12 to R47, R27 to R48, R13 to R49, R28 to R50, R14 to R51, R15 to R52, R29 to R53, V1 to V2, V2 to V3, V3 to V5, V5 to V6, VBOGUS1 to VBOGUS2
Connections:
- net 0: now also C7.1, Q11.3 (E), Q12.3 (E), R1.1, R12.1, R14.1, R26.1, R27.1, R31.1, R36.1, R4.1, R41.1, R42.1, R59.1, R6.1, R60.1, R65.1, R8.1, V1.2, V7.2
- net AUX11-TGL: now also C5.1, R54.1
- net AUX12-TGL: now also C4.1, C6.1
- net E24-12V: now also Q1.1 (C), R11.2, R13.2, R2.2, R5.2, R58.2, R7.2
- net at C2.2, Q6.2 (B), R35.2: now also D9.2 (K); no longer D1.2 (K)
- net at D1.1 (A): now also R2.1, R3.2; no longer R22.1
- new net: C8.2, D13.2 (K), R54.2, R55.2
- new net: R55.1, R56.1
- new net: C7.2, D13.1 (A), R56.2
- new net: C8.1, R57.1
- new net: R10.1, R57.2, R58.1, R59.2
- new net: D1.2 (K), R1.2
- new net: Q1.2 (B), R3.1
- new net: D2.2 (K), R5.1, R6.2, R9.2
- new net: D3.2 (K), R10.2, R7.1, R8.2
- new net: Q2.2 (B), R11.1, R12.2, R9.1
- new net: D9.1 (A), R22.1
- new net: Q2.3 (E), R13.1
- new net: Q2.1 (C), R14.2, R24.2
- new net: C3.2, D10.2 (K), R24.1
- new net: D10.1 (A), R27.2
- new net: C3.1, D11.1 (A), R36.2
- new net: C6.2, D11.2 (K), D12.2 (K)
- new net: D12.1 (A), R41.2, R42.2
- new net: C4.2, D4.2 (K), R30.1, R31.2
- new net: C5.2, D5.2 (K), R25.1, R26.2
- new net: V1.1, VBOGUS1.1
- new net: D16.2 (K), Q11.2 (B), R65.2, R68.2
- new net: C9.2, R68.1
- new net: C9.1, Q12.2 (B), R67.1
- new net: D14.2 (K), R63.2
- new net: D14.1 (A), R61.1, R62.1
- new net: L1.2, R70.1
- new net: L2.1, R71.1
- new net AUX1-10V: R23.2, R25.2, R30.2, R62.2, R64.2, R66.2, R69.2, VBOGUS1.2
- new net AUX10-SP: Q11.1 (C), R66.1, R67.2
- new net AUX9-BP: L1.1, Q12.1 (C), R69.1
- new net E1-T1: R60.2, R61.2
- new net E10-MPS: R71.2, V7.1
- new net E15-MPS: R63.1, R64.1, R70.2
- new net E8-MPS: D15.2 (K), L2.2
- new net EDGES: D15.1 (A), D16.1 (A), D4.1 (A), D5.1 (A), R23.1
- new net WATER-TEMP-BIAS: D2.1 (A), D3.1 (A), Q1.3 (E), R4.2
Other:
- note added: ".model DIODE D\n.model BCY58 npn\n.model BSX95 npn\n.model AUY21 pnp\nL1 1 2 395m\nL2 2 1 792m\nK1 L1 L2 1.0\n.tran 0.01ms 600ms 120m\n.control\nrun\nrusage\nset filetype=ascii\nset color0=white\nset xbrushwidth=5\nwrite "C:\Users\andy\OneDrive\Documents\MPS Tune-o-Matic\trunk\Simulation\Pressure Loop\PressureLoop.out" "V(E22-PG)" "V(E21-PG)" "V(E14-PG)" "V(E13-PG)" "V(INT-7)"\nplot "V(E22-PG)"+5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"
- note added: "Air temp sensor"
- note removed: ".model DIODE D\n.model BCY58 npn\n.model BSX95 npn\n.model AUY21 pnp\n.tran 1ms 600ms 120m\n.control\nrun\nrusage\nset filetype=ascii\nset color0=white\nset xbrushwidth=5\nwrite "C:\Users\andy\OneDrive\Documents\MPS Tune-o-Matic\trunk\Simulation\Pressure Loop\PressureLoop.out" "V(E22-PG)" "V(E21-PG)" "V(E14-PG)" "V(E13-PG)" "V(INT-7)"\nplot "V(E22-PG)"+5 "V(E14-PG)"+10 "V(E21-PG)"+15 "V(E13-PG)"+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"
- moved on the sheet: D1, Q10, Q8, R48, R50, R53, V2, V3, V4, V5, V6, VBOGUS2

Commit message: Wprking on simulation of pressure loop.
Parts:
- removed C3: 33n, Right D Line, symbol Device:C
- removed C6: 470n, Right D Line, symbol Device:C
- removed D1, D10, D11, D12, D2, D3: DIODE, symbol Simulation_SPICE:DIODE
- removed Q1: BCY58, Package_TO_SOT_THT:TO-92_Inline, symbol Transistor_BJT:BC547
- removed Q2: AUY21, symbol Device:Q_PNP_CBE
- removed R1: 100k, Upper Center K, symbol Device:R_US
- removed R10: 510k, Upper Center K, symbol Device:R_US
- removed R11, R7: 22k, Upper Center K, symbol Device:R_US
- removed R12: 68k, Upper Center K, symbol Device:R_US
- removed R13, R14, R24: 10k, Upper Center K, symbol Device:R_US
- removed R2, R4: 1k5, Upper Center K, symbol Device:R_US
- removed R27: 5k6, Upper Center K, symbol Device:R_US
- removed R3: 100, Upper Center K, symbol Device:R_US
- removed R36: 9k1, Upper Center K, symbol Device:R_US
- removed R41: 270k, Upper Center K, symbol Device:R_US
- removed R42: 75k, Upper Center K, symbol Device:R_US
- removed R5: 15k, Upper Center K, symbol Device:R_US
- removed R6: 2k4, Upper Center K, symbol Device:R_US
- removed R8: 4k8, Upper Center K, symbol Device:R_US
- removed R9: 56k, Upper Center K, symbol Device:R_US
- L1: value 395mH -> 501mH
- L2: value 792mH -> 1.043H
- R60: value 240 -> 200
- R70: value 90.7 -> 92.8
- R71: value 340.4 -> 345.1
- V7: value 2 -> 5; Spice_Model dc(2) -> dc(5.0)
Connections:
- net AUX9-BP renamed BASE_PULSE
Other:
- note added: ".model DIODE D\n.model BCY58 npn\n.model BSX95 npn\n.model AUY21 pnp\nL1 1 2 501m\nL2 2 1 1.043H\nK1 L1 L2 1.0\n.tran 0.05ms 600ms 120m\n.control\nrun\nrusage\nset filetype=ascii\nset color0=white\nset xbrushwidth=5\nwrite "C:\Users\andy\OneDrive\Documents\MPS Tune-o-Matic\trunk\Simulation\Pressure Loop\PressureLoop.out" "V(E22-PG)" "V(E21-PG)" "V(E14-PG)" "V(E13-PG)" "V(INT-7)"\nplot "V(E22-PG)"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"
- note removed: ".model DIODE D\n.model BCY58 npn\n.model BSX95 npn\n.model AUY21 pnp\nL1 1 2 395m\nL2 2 1 792m\nK1 L1 L2 1.0\n.tran 0.01ms 600ms 120m\n.control\nrun\nrusage\nset filetype=ascii\nset color0=white\nset xbrushwidth=5\nwrite "C:\Users\andy\OneDrive\Documents\MPS Tune-o-Matic\trunk\Simulation\Pressure Loop\PressureLoop.out" "V(E22-PG)" "V(E21-PG)" "V(E14-PG)" "V(E13-PG)" "V(INT-7)"\nplot "V(E22-PG)"+5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"
- moved on the sheet: C4, C5, C7, C8, D13, D4, D5, Q10, Q8, R23, R25, R26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

Commit message: Using a real coupling factor for MPS.
Other:
- note added: ".model DIODE D\n.model BCY58 npn\n.model BSX95 npn\n.model AUY21 pnp\nL1 1 2 501m\nL2 2 1 1.043H\nK1 L1 L2 0.498\n.tran 0.05ms 600ms 120m\n.control\nrun\nrusage\nset filetype=ascii\nset color0=white\nset xbrushwidth=5\nwrite "C:\Users\andy\OneDrive\Documents\MPS Tune-o-Matic\trunk\Simulation\Pressure Loop\PressureLoop.out" "V(E22-PG)" "V(E21-PG)" "V(E14-PG)" "V(E13-PG)" "V(INT-7)"\nplot "V(E22-PG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"
- note added: "For external ngspice for simulation see: http://ngspice.sourceforge.net/ngspice-eeschema.html, section 6"
- note added: "MPS coupling factor (k) is set to 0.498, which was obtained by measurement with no vacuum"
- note removed: ".model DIODE D\n.model BCY58 npn\n.model BSX95 npn\n.model AUY21 pnp\nL1 1 2 501m\nL2 2 1 1.043H\nK1 L1 L2 1.0\n.tran 0.05ms 600ms 120m\n.control\nrun\nrusage\nset filetype=ascii\nset color0=white\nset xbrushwidth=5\nwrite "C:\Users\andy\OneDrive\Documents\MPS Tune-o-Matic\trunk\Simulation\Pressure Loop\PressureLoop.out" "V(E22-PG)" "V(E21-PG)" "V(E14-PG)" "V(E13-PG)" "V(INT-7)"\nplot "V(E22-PG)"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"
- note removed: "This requires external ngspice for simulation. See:\nhttp://ngspice.sourceforge.net/ngspice-eeschema.html\nsection 6"
- moved on the sheet: C1, C2, D6, D7, D8, D9, Q3, Q4, Q5, Q6, Q7, Q9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

Commit message: Added component for MPS.
Parts:
- removed L1: 501mH, symbol pspice:INDUCTOR
- removed L2: 1.043H, symbol pspice:INDUCTOR
- removed R70: 92.8, Upper Center K, symbol Device:R_US
- removed R71: 345.1, Upper Center K, symbol Device:R_US
- added TR1: MPS, symbol BritishIdeas:MPS
- V7: value 5 -> 4; Spice_Model dc(5.0) -> dc(4.0)
Connections:
- net BASE_PULSE: now also TR1.1 (7_PRI)
- net E10-MPS: now also TR1.4 (10_SEC)
- net E15-MPS: now also TR1.2 (15_PRI)
- net E8-MPS: now also TR1.3 (8_SEC)
Other:
- note added: ".model DIODE D\n.model BCY58 npn\n.model BSX95 npn\n.model AUY21 pnp\n.tran 0.05ms 92ms 89m\n.control\nrun\nrusage\nset filetype=ascii\nset color0=white\nset xbrushwidth=5\nwrite "C:\Users\andy\OneDrive\Documents\MPS Tune-o-Matic\trunk\Simulation\Pressure Loop\PressureLoop.out" "V(BASE_PULSE)" "V(INT-7)"\nplot "V(BASE_PULSE)" "V(INT-7)"\n.endc\n"
- note removed: ".model DIODE D\n.model BCY58 npn\n.model BSX95 npn\n.model AUY21 pnp\nL1 1 2 501m\nL2 2 1 1.043H\nK1 L1 L2 0.498\n.tran 0.05ms 600ms 120m\n.control\nrun\nrusage\nset filetype=ascii\nset color0=white\nset xbrushwidth=5\nwrite "C:\Users\andy\OneDrive\Documents\MPS Tune-o-Matic\trunk\Simulation\Pressure Loop\PressureLoop.out" "V(E22-PG)" "V(E21-PG)" "V(E14-PG)" "V(E13-PG)" "V(INT-7)"\nplot "V(E22-PG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"
Changed lines of the file:
@@
 Comment4 "Main Board 2 288 300 028"
 $EndDescr
-Text Notes 1350 6950 0    50   ~ 0
-.model DIODE D\n.model BCY58 npn\n.model BSX95 npn\n.model AUY21 pnp\nL1 1 2 501m\nL2 2 1 1.043H\nK1 L1 L2 0.498\n.tran 0.05ms 600ms 120m\n.control\nrun\nrusage\nset filetype=ascii\nset color0=white\nset xbrushwidth=5\nwrite "C:\Users\andy\OneDrive\Documents\MPS Tune-o-Matic\trunk\Simulation\Pressure Loop\PressureLoop.out" "V(E22-PG)" "V(E21-PG)" "V(E14-PG)" "V(E13-PG)" "V(INT-7)"\nplot "V(E22-PG)"+5 "V(E14-PG)"+10 "V(E21-PG)"+15 "V(E13-PG)"+20 "V(INT-7)"\n.endc\n
 Text GLabel 2650 4750 3    50   UnSpc ~ 0
 E11-GND
@@
 Wire Wire Line
 	1950 3350 1950 3000
-Wire Wire Line
-	5950 12750 5850 12750
 Text GLabel 5850 12750 0    50   Input ~ 0
 E15-MPS
@@
 P 1300 4250
 F 0 "V7" H 1430 4341 50  0000 L CNN
-F 1 "5" H 1430 4250 50  0000 L CNN
+F 1 "4" H 1430 4250 50  0000 L CNN
 F 2 "" H 1300 4250 50  0001 C CNN
 F 3 "~" H 1300 4250 50  0001 C CNN
 F 4 "Y" H 1300 4250 50  0001 L CNN "Spice_Netlist_Enabled"
 F 5 "V" H 1300 4250 50  0001 L CNN "Spice_Primitive"
-F 6 "dc(5.0)" H 1430 4159 50  0000 L CNN "Spice_Model"
+F 6 "dc(4.0)" H 1430 4159 50  0000 L CNN "Spice_Model"
 	1    1300 4250
 	1    0    0    -1
@@
 Wire Wire Line
 	1300 4050 1300 2950
-Wire Wire Line
-	6750 13450 7400 13450
-$Comp
-L Device:R_US R70
-U 1 1 62996BC8
-P 6100 12750
-F 0 "R70" V 6000 12700 50  0000 L CNN
-F 1 "92.8" V 6200 12600 50  0000 L CNN
-F 2 "Upper Center K" V 6140 12740 50  0001 C CNN
-F 3 "~" H 6100 12750 50  0001 C CNN
-F 4 "O Bk Br Gd = 300Ω ±5%" H 6100 12750 50  0001 C CNN "Notes"
-	1    6100 12750
-	0    1    1    0
-$EndComp
-$Comp
-L Device:R_US R71
-U 1 1 6299740F
-P 6100 13450
-F 0 "R71" V 6200 13400 50  0000 L CNN
-F 1 "345.1" V 6000 13350 50  0000 L CNN
-F 2 "Upper Center K" V 6140 13440 50  0001 C CNN
-F 3 "~" H 6100 13450 50  0001 C CNN
-F 4 "O Bk Br Gd = 300Ω ±5%" H 6100 13450 50  0001 C CNN "Notes"
-	1    6100 13450
-	0    1    1    0
-$EndComp
-Wire Wire Line
-	6750 12750 9950 12750
-Wire Wire Line
-	5700 13450 5950 13450
 Connection ~ 5700 13450
 Wire Wire Line
@@
 Wire Wire Line
 	5600 13450 5700 13450
-$Comp
-L pspice:INDUCTOR L1
-U 1 1 62AE9102
-P 6500 12750
-F 0 "L1" H 6500 12569 50  0000 C CNN
-F 1 "501mH" H 6500 12660 50  0000 C CNN
-F 2 "" H 6500 12750 50  0001 C CNN
-F 3 "~" H 6500 12750 50  0001 C CNN
-	1    6500 12750
-	-1   0    0    1
-$EndComp
-$Comp
-L pspice:INDUCTOR L2
-U 1 1 62B102AA
-P 6500 13450
-F 0 "L2" H 6500 13665 50  0000 C CNN
-F 1 "1.043H" H 6500 13574 50  0000 C CNN
-F 2 "" H 6500 13450 50  0001 C CNN
-F 3 "~" H 6500 13450 50  0001 C CNN
-	1    6500 13450
-	1    0    0    -1
-$EndComp
 Wire Wire Line
 	3700 14300 8350 14300
@@
 	5850 11850 8750 11850
 Connection ~ 8750 11850
-Wire Notes Line
-	6800 12450 6800 13700
-Wire Notes Line
-	6800 13700 5900 13700
-Wire Notes Line
-	5900 13700 5900 12450
-Wire Notes Line
-	5900 12450 6800 12450
 Text Notes 2900 12700 0    50   ~ 0
 Air temp sensor
@@
 Text Notes 1100 1400 0    118  ~ 0
 MPS coupling factor (k) is set to 0.498, which was obtained by measurement with no vacuum
+Text Notes 1350 6950 0    50   ~ 0
+.model DIODE D\n.model BCY58 npn\n.model BSX95 npn\n.model AUY21 pnp\n.tran 0.05ms 92ms 89m\n.control\nrun\nrusage\nset filetype=ascii\nset color0=white\nset xbrushwidth=5\nwrite "C:\Users\andy\OneDrive\Documents\MPS Tune-o-Matic\trunk\Simulation\Pressure Loop\PressureLoop.out" "V(BASE_PULSE)" "V(INT-7)"\nplot "V(BASE_PULSE)" "V(INT-7)"\n.endc\n
+$Comp
+L BritishIdeas:MPS TR1
+U 1 1 61BF306A
+P 6350 13100
+F 0 "TR1" V 6800 12800 50  0000 L CNN
+F 1 "MPS" V 6800 13150 50  0000 L CNN
+F 2 "" H 6350 13100 50  0001 C CNN
+F 3 "" H 6350 13100 50  0001 C CNN
+F 4 "X" H 6350 13100 50  0001 C CNN "Spice_Primitive"
+F 5 "mps1" V 6900 13050 50  0000 C CNN "Spice_Model"
+F 6 "Y" H 6350 13100 50  0001 C CNN "Spice_Netlist_Enabled"
+F 7 "MPS.lib" H 6350 13100 50  0001 C CNN "Spice_Lib_File"
+	1    6350 13100
+	0    1    1    0
+$EndComp
+Wire Wire Line
+	6150 12850 6150 12750
+Wire Wire Line
+	5850 12750 6150 12750
+Wire Wire Line
+	6550 12850 6550 12750
+Wire Wire Line
+	6550 12750 9950 12750
+Wire Wire Line
+	6550 13450 6550 13350
+Wire Wire Line
+	6550 13450 7400 13450
+Wire Wire Line
+	6150 13450 6150 13350
+Wire Wire Line
+	5700 13450 6150 13450
 $EndSCHEMATC

Commit message: Updated MPS model for simulation.
Parts:
- TR1: Spice_Model mps1 -> mps vac=15
Other:
- note added: "Lower voltage = richer"
- note removed: "MPS coupling factor (k) is set to 0.498, which was obtained by measurement with no vacuum"
Changed lines of the file:
@@
 Wire Wire Line
 	13550 7450 17300 7450
-Text Notes 1100 1400 0    118  ~ 0
-MPS coupling factor (k) is set to 0.498, which was obtained by measurement with no vacuum
 Text Notes 1350 6950 0    50   ~ 0
 .model DIODE D\n.model BCY58 npn\n.model BSX95 npn\n.model AUY21 pnp\n.tran 0.05ms 92ms 89m\n.control\nrun\nrusage\nset filetype=ascii\nset color0=white\nset xbrushwidth=5\nwrite "C:\Users\andy\OneDrive\Documents\MPS Tune-o-Matic\trunk\Simulation\Pressure Loop\PressureLoop.out" "V(BASE_PULSE)" "V(INT-7)"\nplot "V(BASE_PULSE)" "V(INT-7)"\n.endc\n
-$Comp
-L BritishIdeas:MPS TR1
-U 1 1 61BF306A
-P 6350 13100
-F 0 "TR1" V 6800 12800 50  0000 L CNN
-F 1 "MPS" V 6800 13150 50  0000 L CNN
-F 2 "" H 6350 13100 50  0001 C CNN
-F 3 "" H 6350 13100 50  0001 C CNN
-F 4 "X" H 6350 13100 50  0001 C CNN "Spice_Primitive"
-F 5 "mps1" V 6900 13050 50  0000 C CNN "Spice_Model"
-F 6 "Y" H 6350 13100 50  0001 C CNN "Spice_Netlist_Enabled"
-F 7 "MPS.lib" H 6350 13100 50  0001 C CNN "Spice_Lib_File"
-	1    6350 13100
-	0    1    1    0
-$EndComp
 Wire Wire Line
 	6150 12850 6150 12750
@@
 Wire Wire Line
 	5700 13450 6150 13450
+$Comp
+L BritishIdeas:MPS TR1
+U 1 1 620F2499
+P 6350 13100
+F 0 "TR1" V 6050 13050 50  0000 L CNN
+F 1 "MPS" V 6600 13000 50  0000 L CNN
+F 2 "" H 6350 13100 50  0001 C CNN
+F 3 "" H 6350 13100 50  0001 C CNN
+F 4 "X" H 6350 13100 50  0001 C CNN "Spice_Primitive"
+F 5 "mps vac=15" V 6800 13100 50  0000 C CNN "Spice_Model"
+F 6 "Y" H 6350 13100 50  0001 C CNN "Spice_Netlist_Enabled"
+F 7 "MPS.lib" H 6350 13100 50  0001 C CNN "Spice_Lib_File"
+	1    6350 13100
+	0    1    1    0
+$EndComp
+Text Notes 850  4700 0    50   ~ 0
+Lower voltage = richer
 $EndSCHEMATC
